File: hw/USB_module.brd (EAGLE design)
At the start: 25 x 45 mm, 45 parts, among them J1 GROVE-4P-2.0-3470130P1, J2 GROVE-4P-2.0-3470130P1, X1 22-23-2021, X2 47589-0001, X4 53047-04, X5 53047-04, X6 53047-06

Commit message: updated USB R value
Parts:
- R8: value 22 -> 1k5
Changed lines of the file:
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@@
 <?xml version="1.0" encoding="utf-8"?>
 <!DOCTYPE eagle SYSTEM "eagle.dtd">
-<eagle version="6.6.0">
+<eagle version="6.4">
 <drawing>
 <settings>
@@
 <element name="R7" library="rcl" package="R0603" value="1k" x="14" y="26.8" rot="R180"/>
 <element name="D6" library="dp_devices" package="SOD-323F" value="3V" x="14.1" y="25.2"/>
-<element name="R8" library="rcl" package="R0603" value="22" x="5.2" y="36.2" rot="R90"/>
+<element name="R8" library="rcl" package="R0603" value="1k5" x="5.2" y="36.2" rot="R90"/>
 <element name="U$7" library="texas-instruments" package="SOT23-6L" value="LM5050-1" x="12.1" y="34.4"/>
 <element name="D1" library="diode" package="SOD123" value="MBR0520LT" x="12.2" y="40.5" rot="R90"/>

Commit message: layout complete
Parts:
- removed D2: (no value), dp_devices:SOD-323F
- removed D6: 3V, dp_devices:SOD-323F
- removed Q1: (no value), transistor-power:SO-08
- removed R7: 1k, rcl:R0603
- removed TVSD1: SMAJ24A, TVSD:SMA
- removed U$7: LM5050-1, texas-instruments:SOT23-6L
- removed X1: 22-23-2021, con-molex:22-23-2021
- removed X2: 47589-0001, molex:47589-0001
- removed X4: 53047-04, con-molex:53047-04
- removed X6: 53047-06, con-molex:53047-06
- added J3: (no value), OPL-Connector:9+4P-SMD-L16.1*W14.5*H1.85MM
- added J4: MICRO-USB-5P-340015001, OPL Eagle Library:B-SMD-5P
- added LED2: (no value), led:CHIPLED_0805
- added R9: 100k, rcl:R0603
- C10: value (none) -> 100n; device rcl:C0805 -> rcl:C0603
- C11: value 10nF -> 4.7u; device rcl:C0603 -> rcl:C0805
- C12: device rcl:E3,5-8 -> rcl:B/3528-21R
- R4: value 4k7 -> 100k
- R5: value (none) -> 100k
- R6: value 10k -> 330
- moved R11 19.0 mm to (7.80, 17.2)
- moved R14 19.0 mm to (6.40, 17.2)
- moved R8 19.0 mm to (5.00, 17.2)
- moved D1 16.3 mm to (22.0, 27.5), turned to 180 degrees
- moved R2 16.0 mm to (5.00, 20.2)
- moved R4 11.6 mm to (17.0, 27.5), turned to 270 degrees
- moved R6 8.10 mm to (22.0, 29.5), turned to 180 degrees
- moved C10 6.83 mm to (13.0, 27.5), turned to 270 degrees
- moved X5 4.88 mm to (14.8, 23.5), turned to 0 degrees
- moved C11 3.57 mm to (14.7, 27.5), turned to 270 degrees
- moved R5 3.26 mm to (11.5, 27.5), turned to 270 degrees
- moved C12 2.06 mm to (22.0, 24.5), turned to 0 degrees
Connections:
- removed net !CS: U$6.25, X6.3
- removed net MISO: U$6.27, X6.5
- removed net MOSI: U$6.28, X6.6
- removed net N$10: C11.1, R5.1, U$7.1
- removed net N$9: Q1.4, U$7.5
- removed net SCK: U$6.26, X6.4
- removed net SCL: U$6.30, X4.3
- removed net SDA: U$6.31, X4.4
- removed net VBATT: C10.2, Q1.1, Q1.2, Q1.3, TVSD1.C, U$7.4, X1.1
- new net SD_!CD: J3.9, U$6.14
- new net SD_!CS: J3.2, R9.1, U$6.25
- new net SD_CLK: J3.5, U$6.26
- new net SD_LED: R6.2, U$6.13
- new net SD_MISO: J3.7, R4.1, U$6.27
- new net SD_MOSI: J3.3, R5.1, U$6.28
- net +3V3: now also C10.1, C11.1, J3.4, R4.2, R5.2, R9.2; no longer X4.1, X6.1
- net GND: now also C10.2, J3.6, J4.5, J4.E1, J4.E2, J4.P1, J4.P2, LED2.A; no longer C10.1, D2.A, D6.A, R7.1, TVSD1.A, U$7.2, X1.2, X2.5, X2.SHLD1, X2.SHLD2, X2.SHLD3, X2.SHLD4, X4.2, X6.2
- net N$3: now also J4.2; no longer X2.2
- net N$32: now also J4.3; no longer X2.3
- net N$5: now also J4.4; no longer X2.4
- net N$6: now also LED2.C, R6.1; no longer D2.C, R4.1, U$7.3
- net USB_VBUS: now also J4.1; no longer R4.2, X2.1
- net VIN: no longer Q1.5, Q1.6, Q1.7, Q1.8, R5.2, R6.2, U$7.6
- net VSENSE: no longer D6.C, R6.1, R7.2
Routing:
- net VIN: track 66.4 -> 42.9 mm, vias 2 -> 1
- net USB_N: track 24.6 -> 3.00 mm
- net USB_P: track 24.9 -> 4.93 mm
- net SD_MOSI: track 0.00 -> 18.8 mm, vias 0 -> 2
- net SD_MISO: track 0.00 -> 18.5 mm, vias 0 -> 2
- net SD_!CS: track 0.00 -> 15.5 mm, vias 0 -> 2
- net SD_CLK: track 0.00 -> 14.5 mm, vias 0 -> 2
- net !CS: track 14.4 -> 0.00 mm, vias 1 -> 0
- net SCK: track 13.7 -> 0.00 mm, vias 1 -> 0
- net MISO: track 12.7 -> 0.00 mm, vias 1 -> 0
- net MOSI: track 11.9 -> 0.00 mm, vias 1 -> 0
- net SCL: track 11.4 -> 0.00 mm
- net SD_LED: track 0.00 -> 11.4 mm
- net SD_!CD: track 0.00 -> 11.1 mm
- net SDA: track 10.3 -> 0.00 mm
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- removed copper zone on layer 1, net VBATT
Other:
- board text removed: "I2C"
- board text removed: "SPI"

Commit message: layout completed
Parts:
- R4, R5, R9: value 100k -> 47k
- moved C12 0.50 mm to (21.5, 24.5)
- moved D1 0.50 mm to (21.5, 27.5)
Changed lines of the file:
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@@
 <element name="R2" library="rcl" package="R0603" value="100k" x="5" y="20.2" rot="R90"/>
 <element name="R8" library="rcl" package="R0603" value="1k5" x="5" y="17.2" rot="R90"/>
-<element name="D1" library="diode" package="SOD123" value="MBR0520LT" x="22" y="27.5" rot="R180"/>
+<element name="D1" library="diode" package="SOD123" value="MBR0520LT" x="21.5" y="27.5" rot="R180"/>
 <element name="J3" library="OPL-Connector" package="9+4P-SMD-L16.1*W14.5*H1.85MM" value="" x="12.5" y="31" rot="R90"/>
-<element name="R4" library="rcl" package="R0603" value="100k" x="17" y="27.5" rot="R270"/>
-<element name="R5" library="rcl" package="R0603" value="100k" x="11.5" y="27.5" rot="R270"/>
-<element name="R9" library="rcl" package="R0603" value="100k" x="9.7" y="27.5" rot="R270"/>
+<element name="R4" library="rcl" package="R0603" value="47k" x="17" y="27.5" rot="R270"/>
+<element name="R5" library="rcl" package="R0603" value="47k" x="11.5" y="27.5" rot="R270"/>
+<element name="R9" library="rcl" package="R0603" value="47k" x="9.7" y="27.5" rot="R270"/>
 <element name="J4" library="OPL Eagle Library" package="B-SMD-5P" value="MICRO-USB-5P-340015001" x="2.5" y="26" rot="R270"/>
 <element name="C10" library="rcl" package="C0603" value="100n" x="13" y="27.5" rot="R270"/>
 <element name="C11" library="rcl" package="C0805" value="4.7u" x="14.7" y="27.5" rot="R270"/>
-<element name="C12" library="rcl" package="B/3528-21R" value="" x="22" y="24.5"/>
+<element name="C12" library="rcl" package="B/3528-21R" value="" x="21.5" y="24.5"/>
 <element name="LED2" library="led" package="CHIPLED_0805" value="" x="23" y="42.5" rot="R180"/>
 <element name="R6" library="rcl" package="R0603" value="330" x="22" y="29.5" rot="R180"/>
@@
 <contactref element="C12" pad="+"/>
 <via x="23.9" y="21.878" extent="1-16" drill="0.6"/>
-<wire x1="23.9" y1="21.878" x2="23.525" y2="22.253" width="1" layer="1"/>
-<wire x1="23.525" y1="22.253" x2="23.525" y2="24.5" width="1" layer="1"/>
-<wire x1="23.525" y1="24.5" x2="23.9" y2="24.875" width="1" layer="1"/>
-<wire x1="23.9" y1="24.875" x2="23.9" y2="27.5" width="1" layer="1"/>
+<wire x1="23.9" y1="21.878" x2="23.025" y2="22.753" width="1" layer="1"/>
+<wire x1="23.025" y1="22.753" x2="23.025" y2="24.5" width="1" layer="1"/>
+<wire x1="23.025" y1="24.5" x2="23.4" y2="24.875" width="1" layer="1"/>
+<wire x1="23.4" y1="24.875" x2="23.4" y2="27.5" width="1" layer="1"/>
 </signal>
 <signal name="+3V3">
@@
 <wire x1="5.04" y1="27.3" x2="6.4" y2="27.3" width="0.4" layer="1"/>
 <wire x1="6.4" y1="27.3" x2="10.6" y2="31.5" width="1" layer="16"/>
-<wire x1="10.6" y1="31.5" x2="17.5" y2="31.5" width="1" layer="16"/>
-<via x="20.1" y="28.5" extent="1-16" drill="0.3"/>
-<wire x1="20.1" y1="28.5" x2="20.1" y2="27.5" width="1" layer="1"/>
-<wire x1="17.5" y1="31.5" x2="20.1" y2="28.9" width="1" layer="16"/>
-<wire x1="20.1" y1="28.9" x2="20.1" y2="28.5" width="1" layer="16"/>
+<wire x1="10.6" y1="31.5" x2="17.6" y2="31.5" width="1" layer="16"/>
+<via x="19.6" y="28.5" extent="1-16" drill="0.3"/>
+<wire x1="19.6" y1="28.5" x2="19.6" y2="27.5" width="1" layer="1"/>
+<wire x1="17.6" y1="31.5" x2="19.6" y2="29.5" width="1" layer="16"/>
+<wire x1="19.6" y1="29.5" x2="19.6" y2="28.5" width="1" layer="16"/>
 </signal>
 <signal name="USB_N">
